File: led_array.kicad_sch (KiCad schematic)
At the start: 3 parts, among them U6 74AHCT1G125

Commit message: Final schematic before review.
Parts:
- renumbered D2 to D1, U6 to U5
Changed lines of the file:
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@@
 		(dnp yes)
 		(fields_autoplaced yes)
-		(property "Reference" "D2"
+		(property "Reference" "D1"
 			(at 170.18 41.8398 0)
 			(effects
@@
 			(project "universal-board"
 				(path "/64404f27-cfd6-41d9-8edb-810ebab8cc14/b28a21dd-1aff-4e24-a93f-dbc2ef34d4d1"
-					(reference "D2")
+					(reference "D1")
 					(unit 1)
 				)
@@
 		(dnp no)
 		(fields_autoplaced yes)
-		(property "Reference" "U6"
+		(property "Reference" "U5"
 			(at 109.22 41.8398 0)
 			(effects
@@
 			(project "universal-board"
 				(path "/64404f27-cfd6-41d9-8edb-810ebab8cc14/b28a21dd-1aff-4e24-a93f-dbc2ef34d4d1"
-					(reference "U6")
+					(reference "U5")
 					(unit 1)
 				)
